File: PCB.sch (EAGLE design)
At the start: 27 parts, among them P1.0 WIREPAD1,6/0,9, P1.3 WIREPAD1,6/0,9, P1.4 WIREPAD1,6/0,9, P2.2 WIREPAD1,6/0,9, P2.7 WIREPAD1,6/0,9, U1 MSP430G2553_PW_20, U2 DRV8833_PWP_16, U3 DRV8833_PWP_16

Commit message: Magor version revision
Fixed timer pinout problem
updated silk screen with new logo
broke out power and data to different headers
reworked MCU power isolation
Parts:
- removed JP1: (no value), jumper:JP4E
- added D2: (no value), adafruit:DIODESOD-123
- added JP3: (no value), jumper:JP1E
- added POWER: 22-23-2021, con-molex:22-23-2021
- added R6: (no value), adafruit:R-US_R1206
- D1: device adafruit:DIODESMA -> adafruit:DIODESOD-123
- R1, R2, R3, R4, R5: device adafruit:R-US_0204/2V -> adafruit:R-US_R1206
- renumbered P1.4 to P2.6, P2.2 to P2.3
Connections:
- removed net P1.4: P2.6.P, U1.P1.4/SMCLK/UCB0STE/UCA0CLK/VREF+/VEREF+/A4/CA4/TCK
- removed net P2.2: P2.3.P, U1.P2.2/TA1.1
- new net +3V3UNREG: D1.C, R6.1
- new net P2.3: P2.3.P, U1.P2.3/TA1.0
- new net P2.6: P2.6.P, U1.XIN/P2.6/TA0.1
- net +3V3: now also D2.C, R6.2; no longer D1.C
- net +3V3MOTOR: now also POWER-2.S; no longer JP1.4
- net GND: now also D2.A, POWER-1.S; no longer JP1.1
- net N1ERROR: now also U1.P2.0/TA1.0; no longer U1.P2.4/TA1.2
- net N1IN1: now also U1.P2.1/TA1.1; no longer U1.P1.5/TA0.0/UCB0CLK/UCA0STE/A5/CA5/TMS
- net N1IN2: now also U1.P2.2/TA1.1; no longer U1.XIN/P2.6/TA0.1
- net N2ERROR: now also U1.P1.4/SMCLK/UCB0STE/UCA0CLK/VREF+/VEREF+/A4/CA4/TCK; no longer U1.P2.3/TA1.0
- net N2IN1: now also U1.P2.4/TA1.2; no longer U1.P2.0/TA1.0
- net N2IN2: now also U1.P2.5/TA1.2; no longer U1.P2.1/TA1.1
- net NRESET: now also U1.P1.5/TA0.0/UCB0CLK/UCA0STE/A5/CA5/TMS; no longer U1.P2.5/TA1.2
- net SCL: now also JP3.1; no longer JP1.2
- net SDA: now also JP3.2; no longer JP1.3
Other:
- moved on the sheet: D1

Commit message: Updated power managment
Added LDO for mcu power
Added buffered voltage divider to allow mcu to measure rail voltage
Repurposed P1.0 to measure rail voltage
Parts:
- removed D2: (no value), adafruit:DIODESOD-123
- removed P1.0: WIREPAD1,6/0,9, wirepad:WIREPAD1,6/0,9
- added C10, C9: (no value), adafruit:C-USC1206
- added R7: 250k, adafruit:R-US_R1206
- added U4: REG101-3_DBV_5, TI:REG101-3_DBV_5
- added U6: TLV2241_DBV_5, TI:TLV2241_DBV_5
- R6: value (none) -> 500k
Connections:
- removed net +3V3MOTOR: C4.2, C5.1, C7.2, C8.1, D1.A, POWER-2.S, U2.VM, U3.VM
- removed net +3V3UNREG: D1.C, R6.1
- removed net P1.0: P1.0.P, U1.P1.0/TA0CLK/ACLK/A0/CA0
- new net 3VOUT: D1.A, U4.VOUT
- new net N$1: C9.2, U4.NR/ADJUST
- new net VCC: C10.1, C4.2, C5.1, C7.2, C8.1, POWER-2.S, R6.2, U2.VM, U3.VM, U4.ENABLE, U4.VIN
- new net VSENSE_IN: R6.1, R7.2, U6.IN+
- new net VSENSE_OUT: U1.P1.0/TA0CLK/ACLK/A0/CA0, U6.IN-, U6.OUT
- net +3V3: now also D1.C, U6.VCC; no longer D2.C, R6.2
- net GND: now also C10.2, C9.1, R7.1, U4.GND, U6.GND; no longer D2.A
Other:
- note added: "MCU/LOGIC POWER"
- note added: "VOLTAGE MEASUREMENT"
- moved on the sheet: D1, POWER-1, POWER-2, R6
