File: PCB.sch (EAGLE design)
At the start: 27 parts, among them P1.0 WIREPAD1,6/0,9, P1.3 WIREPAD1,6/0,9, P1.4 WIREPAD1,6/0,9, P2.2 WIREPAD1,6/0,9, P2.7 WIREPAD1,6/0,9, U1 MSP430G2553_PW_20, U2 DRV8833_PWP_16, U3 DRV8833_PWP_16

Commit message: added power board and gitignore
Parts:
- removed C2: 1 nF, adafruit:C-USC1206
- removed D1: (no value), adafruit:DIODESMA
- removed JP1: (no value), jumper:JP4E
- removed JP2: (no value), jumper:JP1E
- removed P1.0, P1.3, P1.4, P2.2, P2.7: WIREPAD1,6/0,9, wirepad:WIREPAD1,6/0,9
- removed R3: 200k, adafruit:R-US_0204/2V
- added C10, C11: 23p, adafruit:C-USC1206
- added C12: (no value), adafruit:C-USC0603
- added C9: 2.2n, adafruit:C-USC0603
- added IC1: MCP2515-E/ST, mcp2515:MCP2515-E/ST
- added JP4: (no value), adafruit:PINHD-2X9-BIG
- added POWER, STATUS: (no value), adafruit:LEDCHIP-LED0603
- added Q2: QUARZ5, sMSP430:QUARZ5
- added R7, R8: (no value), adafruit:R-US_R0603
- added U5: MSP430G2553_PW_28, TexasInstruments:MSP430G2553_PW_28
- C1: device adafruit:C-USC1206 -> adafruit:C-USC0603
- ICSP: value (none) -> 6-PIN-ICSPTAGCONNECT-HOLES; device con-lstb:MA04-1 -> LaunchFET:6-PIN-ICSPTAGCONNECT-HOLES
- R1: device adafruit:R-US_0204/2V -> adafruit:R-US_R0603
- R2: value 200k -> 47k; device adafruit:R-US_0204/2V -> adafruit:R-US_R0603
- R4, R5: device adafruit:R-US_0204/2V -> adafruit:R-US_R0805
- U1: value MSP430G2553_PW_20 -> SN65HVD235_D_8; device TI:MSP430G2553_PW_20 -> TexasInstruments:SN65HVD235_D_8
Connections:
- removed net +3V3MOTOR: C4.2, C5.1, C7.2, C8.1, D1.A, JP1.4, U2.VM, U3.VM
- removed net NRESET: U1.P2.5/TA1.2, U2.NSLEEP, U3.NSLEEP
- removed net P1.0: P1.0.P, U1.P1.0/TA0CLK/ACLK/A0/CA0
- removed net P1.3: P1.3.P, U1.P1.3/ADC10CLK/CAOUT/VREF-/VEREF-/A3/CA3
- removed net P1.4: P1.4.P, U1.P1.4/SMCLK/UCB0STE/UCA0CLK/VREF+/VEREF+/A4/CA4/TCK
- removed net P2.2: P2.2.P, U1.P2.2/TA1.1
- removed net P2.7: P2.7.P, U1.XOUT/P2.7
- removed net SCL: JP1.2, R3.1, U1.P1.6/TA0.1/UCB0SOMI/UCB0SCL/A6/CA6/TDI/TCLK
- removed net SDA: JP1.3, R2.1, U1.P1.7/CAOUT/UCB0SIMO/UCB0SDA/A7/CA7/TDO/TDI
- new net AUTO_BAUD: U1.AB, U5.P1.3/ADC10CLK/CAOUT/VREF-/VEREF-/A3/CA3
- new net CAN_H: JP4.2, U1.CANH
- new net CAN_L: JP4.3, U1.CANL
- new net CAN_RESET: IC1.RESET, U5.XOUT/P2.7
- new net CLK: IC1.SCK, U5.P1.5/TA0.0/UCB0CLK/UCA0STE/A5/CA5/TMS
- new net EXT_XIN: IC1.CLKOUT, U5.XIN/P2.6/TA0.1
- new net LED0: R1.2, U5.P1.0/TA0CLK/ACLK/A0/CA0
- new net MISO: IC1.SO, U5.P1.6/TA0.1/UCB0SOMI/UCB0SCL/A6/CA6/TDI/TCLK
- new net MOSI: IC1.SI, U5.P1.7/CAOUT/UCB0SIMO/UCB0SDA/A7/CA7/TDO/TDI
- new net N$2: R1.1, STATUS.C
- new net N$5: POWER.C, R7.1
- new net N1RESET: U2.NSLEEP, U5.P2.4/TA1.2
- new net N2RESET: U3.NSLEEP, U5.P2.1/TA1.1
- new net RX0BF: IC1.RX0BF, U5.P2.3/TA1.0
- new net RX1BF: IC1.RX1BF, U5.P3.4/TA0.0
- new net RXINT: IC1.INT, U5.P3.7/TA1CLK/CAOUT
- new net RX_CAN: IC1.RXCAN, U1.R
- new net STE: IC1.CS, U5.P1.4/SMCLK/UCB0STE/UCA0CLK/VREF+/VEREF+/A4/CA4/TCK
- new net TX0RTS: IC1.TX0RTS, U5.P3.1/TA1.0
- new net TX1RTS: IC1.TX1RTS, U5.P3.0/TA0.2
- new net TX2RTS: IC1.TX2RTS, U5.P2.0/TA1.0
- new net TX_CAN: IC1.TXCAN, U1.D
- new net VBUS: C4.2, C5.1, C7.2, C8.1, JP4.11, JP4.13, JP4.15, JP4.17, U2.VM, U3.VM
- new net XIN: C10.1, IC1.OSC1, Q2.2
- new net XOUT: IC1.OSC2, R8.1
- new net XOUT_C: C11.1, Q2.1, R8.2
- net +3V3: now also C12.1, IC1.VDD, ICSP.VCC, JP4.7, JP4.9, POWER.A, STATUS.A, U1.VCC, U5.DVCC; no longer D1.C, ICSP.4, R1.2, R3.2, U1.DVCC
- net GND: now also C10.2, C11.2, C12.2, C9.2, IC1.VSS, ICSP.GND, JP4.1, JP4.12, JP4.14, JP4.16, JP4.18, JP4.4, JP4.5, JP4.6, Q2.0, R7.2, U1.GND, U1.RS, U5.DVSS; no longer C2.2, ICSP.1, JP1.1, U1.DVSS
- net N1ERROR: now also U5.P2.5/TA1.2; no longer U1.P2.4/TA1.2
- net N1IN1: now also U5.P3.5/TA0.1; no longer U1.P1.5/TA0.0/UCB0CLK/UCA0STE/A5/CA5/TMS
- net N1IN2: now also U5.P3.6/TA0.2; no longer U1.XIN/P2.6/TA0.1
- net N2ERROR: now also U5.P2.2/TA1.1; no longer U1.P2.3/TA1.0
- net N2IN1: now also U5.P3.2/TA1.1; no longer U1.P2.0/TA1.0
- net N2IN2: now also U5.P3.3/TA1.2; no longer U1.P2.1/TA1.1
- net RST: now also C9.1, ICSP.RESET, R2.1, U5.*RST/NMI/SBWTDIO; no longer C2.1, ICSP.2, R1.1, U1.*RST/NMI/SBWTDIO
- net TEST: now also ICSP.TEST, U5.TEST/SBWTCK; no longer ICSP.3, U1.TEST/SBWTCK
- net UART_RX: now also ICSP.RX, U5.P1.1/TA0.0/UCA0RXD/UCA0SOMI/A1/CA1; no longer JP2.1, U1.P1.1/TA0.0/UCA0RXD/UCA0SOMI/A1/CA1
- net UART_TX: now also ICSP.TX, U5.P1.2/TA0.1/UCA0TXD/PUCA0SIMO/A2/CA2; no longer JP2.2, U1.P1.2/TA0.1/UCA0TXD/UCA0SIMO/A2/CA2
Other:
- note added: "Reset conditioning"
- moved on the sheet: C1, C3, C4, C5, C6, C7, C8, R1, R2, R4, R5, U2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

Commit message: major topology changes
Parts:
- removed JP4: (no value), adafruit:PINHD-2X9-BIG
- added C2: (no value), adafruit:C-USC0603
- added SV1: (no value), con-lstb:MA05-2
- added U$2: 1X4_HEADER, connectors:1X4_HEADER
- added U$3, U$4: 1X2_HEADER, connectors:1X2_HEADER
Connections:
- removed net VBUS: C4.2, C5.1, C7.2, C8.1, JP4.11, JP4.13, JP4.15, JP4.17, U2.VM, U3.VM
- new net VBUS-M1: C7.2, C8.1, U$2.3, U$2.4, U3.VM
- new net VBUS-M2: C4.2, C5.1, U$4.1, U$4.2, U2.VM
- net +3V3: now also C2.1, SV1.1, SV1.2, SV1.3, SV1.4; no longer JP4.7, JP4.9
- net CAN_H: now also SV1.9; no longer JP4.2
- net CAN_L: now also SV1.8; no longer JP4.3
- net GND: now also C2.2, SV1.10, SV1.5, SV1.6, SV1.7, U$2.1, U$2.2, U$3.1, U$3.2; no longer JP4.1, JP4.12, JP4.14, JP4.16, JP4.18, JP4.4, JP4.5, JP4.6
Other:
- moved on the sheet: C1, C10, C11, C12, C6, C7, C8, C9, IC1, ICSP, POWER, Q2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
