File: power board/base_v2.sch (EAGLE design)
At the start: 59 parts, among them IC1 MCP2515-E/ST, Q2 QUARZ5, U1 INA209_PW_16, U2 LTC1540, U5 MSP430FR5739_DA_38, U6 SN65HVD235_D_8, X1 22-23-2021

Commit message: clean up schematics
Other:
- note added: "Bat Level LEDs"
- note added: "CAN Bus crystal"
- note added: "CAN bus"
- note added: "I2C cond"
- note added: "ICSP"
- note added: "MCU"
- note added: "MCU decoupling"
- note added: "Power/Data Bus out"
- note added: "Status LED"
- moved on the sheet: 100%, 25%, 50%, 75%, C1, C11, C12, C13, C14, C16, C2, C3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
