File: power board/vbus_v2.brd (EAGLE design)
At the start: 60.4 x 36.6 mm, 54 parts, among them U1 LTC1540, U2 TPS70930-Q1, U3 LTC6102, U4 LM45_DBZ_3, U5 MSP430FR5739_DA_38

Commit message: clean up schematics
Parts:
- removed 100%, 25%, 50%, 75%: (no value), adafruit:CHIP-LED0603
- removed C14: 10u, adafruit:C1206
- removed JP1: (no value), jumper:JP1
- removed OA1: LMP2202, TexasInstruments:D8-L
- removed R19, R21, R22, R24: (no value), adafruit:R0603
- added C12: 470n, adafruit:C1206
- added U$1: MICROPITCH, connectors:2X5-1.27MM
- added U$5: MOLEX-0436500200, connectors:MOLEX_MICROFIT-2
- added U6: MSP430FR5739_DA_38, TexasInstruments:DA38
- C1: value 2.2n -> 10u
- C10: value 47uF -> 10u; device rcl:C1206 -> adafruit:C1206
- C11: value .1uF -> 0.1u; device adafruit:C0805 -> adafruit:C1206
- C13: value 10u -> 2.2n
- C2: value 470n -> 10u
- C3: value 10u -> .1uF; device adafruit:C1206 -> adafruit:C0805
- C4: value 0.1u -> .1uF; device adafruit:C1206 -> adafruit:C0805
- C5, C6: value (none) -> 47uF; device adafruit:C0805 -> rcl:C1206
- C8: value .1uF -> (none)
- C9: value 47uF -> (none); device rcl:C1206 -> adafruit:C0805
- R1: value 10k -> 4.8M; device adafruit:M0805 -> adafruit:R1206
- R12: value 100k -> 10k; device adafruit:R1206 -> adafruit:M0805
- R13: value 10k -> 2.3k
- R14: value 2.3k -> 47k; device adafruit:M0805 -> adafruit:R1206
- R15: value 10k -> 1.18M; device adafruit:M0805 -> adafruit:R0805
- R16: value 2.3k -> 1.18M; device adafruit:M0805 -> adafruit:R0805
- R2: value 4.8M -> 1.18M
- R3: value 1.18M -> 100k
- R4: value 47k -> 250R; device adafruit:R1206 -> adafruit:M0805
- R6: value 250R -> 3k
- R7: value 3k -> 10k
- R8: value 1.18M -> 2.3k; device adafruit:R0805 -> adafruit:M0805
- R9: value 1.18M -> 10k; device adafruit:R0805 -> adafruit:M0805
- U4: value LM45_DBZ_3 -> LMP2202; device TexasInstruments:MF03A -> TexasInstruments:D8-L
- U5: value MSP430FR5739_DA_38 -> LM45_DBZ_3; device TexasInstruments:DA38 -> TexasInstruments:MF03A
- moved R14 43.5 mm to (2.89, 7.83), turned to 90 degrees
- moved R12 36.2 mm to (45.1, 22.4), turned to 270 degrees
- moved R9 28.3 mm to (20.5, 31.0), turned to 180 degrees
- moved R15 26.3 mm to (22.8, 1.94), turned to 180 degrees
- moved U5 24.9 mm to (29.4, 29.6), flipped to the bottom, turned to 90 degrees
- moved R4 23.9 mm to (18.5, 28.9), turned to 0 degrees
- moved C1 23.3 mm to (11.8, 29.7), turned to 90 degrees
- moved C13 22.9 mm to (5.18, 7.75)
- moved C2 20.4 mm to (11.2, 22.1), turned to 180 degrees
- moved C3 19.5 mm to (14.9, 31.3), turned to 0 degrees
- moved C9 18.9 mm to (7.62, 28.5)
- moved C10 17.4 mm to (16.5, 17.8), turned to 0 degrees
- moved R16 17.0 mm to (22.8, 4.61), turned to 180 degrees
- moved C6 16.8 mm to (23.6, 33.6)
- moved R8 16.8 mm to (30.2, 19.9), turned to 270 degrees
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- renumbered U$10 to T1, U$12 to T2, U$4 to RSENSE
Connections:
- removed net +3V3_MCU: C3.1, C4.1, R4.2, U$2.VCC
- removed net LED1: R24.2
- removed net LED2: R21.2
- removed net LED3: R22.2
- removed net N$1: 25%.C, R19.1
- removed net N$14: 100%.A, 25%.A, 50%.A, 75%.A
- removed net N$33: 50%.C, R22.1
- removed net N$34: 75%.C, R21.1
- removed net N$35: 100%.C, R24.1
- new net CLK: U$1.10, U6.37
- new net N$13: U$1.4, U6.19
- new net N$16: U$1.8, U6.17
- new net N$19: U$1.5, U6.15
- new net N$20: U$1.3, U6.14
- new net N$21: U$1.1, U6.13
- new net N$22: U$1.6, U6.18
- new net N$24: U$1.2, U6.20
- new net PWM: C9.1, R11.1, U6.12
- new net STE: U$1.9, U6.36
- net +3V3: now also C10.1, C2.1, C4.1, R14.2, R15.1, R16.1, U$2.VCC, U4.8, U5.1, U6.34, U6.4; no longer C14.1, OA1.8, R8.1, R9.1, U4.1, U5.34, U5.4
- net GND: now also C12.2, C5.2, C6.2, R13.2, R2.1, R3.2, R6.2, R8.2, U$5.P$2, U4.4, U6.1, U6.2, U6.25, U6.26, U6.27, U6.28, U6.29, U6.3, U6.33, U6.35, U6.38; no longer C14.2, C3.2, C9.2, JP1.2, OA1.4, R12.2, R14.2, R16.2, R3.1, R7.2, U4.3, U5.33, U5.38
- net I_SENSE: now also R6.1, U6.8; no longer R7.1, U5.11
- net N$11: now also C8.1, R9.2; no longer C5.1, R1.2
- net N$12: now also C9.2; no longer C6.2
- net N$17: now also U$1.7, U6.16; no longer C6.1, R11.1, U5.29
- net N$18: now also C5.1, C6.1, R7.1, R9.1; no longer C10.1, C9.1, R1.1, R15.1
- net N$3: now also R1.1, R2.2; no longer R2.1, R3.2
- net N$4: now also R4.1; no longer R6.1
- net N$6: now also R4.2; no longer R6.2
- net N$7: now also C8.2; no longer C5.2
- net N$8: now also C3.2; no longer C8.2
- net OB_ALERT: now also U6.7; no longer U5.35
- net RST: now also C13.1, R14.1, U6.22; no longer C1.1, R4.1, U5.22
- net SCL: now also R16.2, U6.31; no longer R9.2, U5.31
- net SDA: now also R15.2, U6.30; no longer R8.2, U5.30
- net T1: now also U5.2, U6.10; no longer U4.2, U5.8
- net TEST: now also U6.21; no longer U5.21
- net UART_RX: now also U6.24; no longer U5.24
- net UART_TX: now also U6.23; no longer U5.23
- net VCC: now also C1.1, C3.1, R1.2; no longer C13.1, C8.1, R2.2
- net VCORE: now also C12.1, U6.32; no longer C2.1, U5.32
- net VENABLE: now also R3.1; no longer R12.1
- net V_OUT: now also R12.1, U$5.P$1; no longer JP1.1, R13.1
- net V_SENSE: now also R12.2, R13.1, U4.5; no longer OA1.5, R13.2, R14.1
- net V_SENSE_IN: now also U4.1, U4.2, U6.9; no longer OA1.1, OA1.2, U5.10
- net V_SENSE_IN_P: now also R7.2, R8.1, U4.3; no longer OA1.3, R15.2, R16.1
- net V_SENSE_OUT: now also U4.6, U4.7, U6.11; no longer OA1.6, OA1.7, U5.9
Routing:
- net +3V3: track 50.3 -> 112.8 mm, vias 3 -> 8
- net N$13: track 0.00 -> 39.0 mm, vias 0 -> 3
- net RST: track 3.58 -> 42.3 mm
- net N$22: track 0.00 -> 35.8 mm, vias 0 -> 3
- net N$24: track 0.00 -> 35.7 mm, vias 0 -> 2
- net GND: track 103.1 -> 133.0 mm, vias 6 -> 47
- net N$21: track 0.00 -> 26.6 mm
- net N$16: track 0.00 -> 26.0 mm, vias 0 -> 2
- net N$20: track 0.00 -> 25.5 mm
- net N$19: track 0.00 -> 24.7 mm
- net SDA: track 13.5 -> 36.2 mm, vias 0 -> 1
- net SCL: track 10.4 -> 31.1 mm, vias 0 -> 1
- net PWM: track 0.00 -> 17.8 mm
- net N$17: track 12.4 -> 24.0 mm
- net OB_ALERT: track 0.00 -> 11.6 mm
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Other:
- board size 60.4 x 36.6 mm -> 58.4 x 36.6 mm
