File: power board/vbus_v2.sch (EAGLE design)
At the start: 75 parts, among them IC1 MCP2515-E/ST, Q1 BUZ10, Q2 QUARZ5, U1 INA209_PW_16, U2 UCC2837_D_8, U3 AD5252BRU10, U5 MSP430FR5739_DA_38, U6 SN65HVD235_D_8

Commit message: major topology changes
Parts:
- removed 3V3RAIL, 5VRAIL: (no value), adafruit:LEDCHIP-LED0603
- removed C12: (no value), adafruit:C-USC0603
- removed C15: 68 nF, adafruit:C-USC0805
- removed C16, C17, C18, C19, C20, C21, C22: (no value), adafruit:C-USC0805
- removed C23: 0.1F, adafruit:C-USC0805
- removed C24: .1F, adafruit:C-USC0805
- removed C25: 820pF, adafruit:C-USC0805
- removed C26: 330 F, adafruit:C-USC0805
- removed C27: 1000F, adafruit:C-USC0805
- removed C28: 10uF, adafruit:C-USC0603
- removed IC1: MCP2515-E/ST, mcp2515:MCP2515-E/ST
- removed JP4: (no value), con-lsta:FE05-2
- removed Q1: BUZ10, transistor-fet:BUZ10
- removed Q2: QUARZ5, sMSP430:QUARZ5
- removed R17, R18: (no value), adafruit:R-US_M0805
- removed R23: 10k, adafruit:R-US_M0805
- removed R25: (no value), resistor-shunt:SMR
- removed S1: SWS002, smd-special:SWS002
- removed U$1: LTC3114, linear:LTC3114
- removed U$5: DC630R-562M, connectors:DC630R-562M
- removed U$6: MOLEX_15-31-1026, connectors:MOLEX_15-31-1026
- removed U6: SN65HVD235_D_8, TexasInstruments:SN65HVD235_D_8
- removed X1: (no value), con-wago-500:W237-102
- added D1: UPS840E3/TR13, misc_passives:UPS840E3
- added FET1: P-MOSFET-FDS6681Z, misc_passives:P-MOSFET-FDS6681Z
- added JP1: (no value), jumper:JP1E
- added L1: 10uH, misc_passives:HCF1007
- added OA1: LMP2202, TexasInstruments:LMP2202
- added U$10: NPN-PNP-QSZ4TR, misc_passives:NPN-PNP-QSZ4TR
- added U$11, U$8: 1X4_HEADER, connectors:1X4_HEADER
- added U$12: NPN-2SC5866TLQ, misc_passives:NPN-2SC5866TLQ
- added U4: LM45_DBZ_3, TexasInstruments:LM45_DBZ_3
- C10: value 4.7 pF -> 47uF; device adafruit:C-USC0805 -> rcl:C-EUC1206
- C11: value 4700 pF -> .1uF
- C13: value 68 nF -> 10u; device adafruit:C-USC0805 -> adafruit:C-USC1206
- C14: value 10 uF -> 10u; device adafruit:C-USC0805 -> adafruit:C-USC1206
- C5: value 10u -> (none); device adafruit:C-USC1206 -> adafruit:C-USC0805
- C6: value 33 nF -> (none)
- C7: value 23p -> 47uF; device adafruit:C-USC1206 -> rcl:C-EUC1206
- C8: value 23p -> .1uF; device adafruit:C-USC1206 -> adafruit:C-USC0805
- C9: value 30 uF -> 47uF; device adafruit:C-USC0805 -> rcl:C-EUC1206
- R1: value (none) -> 10k; device resistor-shunt:SMR -> adafruit:R-US_M0805
- R10, R11: value (none) -> 10k; device adafruit:R-US_R0603 -> adafruit:R-US_M0805
- R12: value (none) -> 100k; device adafruit:R-US_M0805 -> adafruit:R-US_R1206
- R13: value 25k -> 10k
- R14: value 27.4k -> 2.3k
- R15: value (none) -> 10k
- R16: value 1.57M -> 2.3k; device adafruit:R-US_R0805 -> adafruit:R-US_M0805
- R2: value 2.25M -> 4.8M; device adafruit:R-US_R0805 -> adafruit:R-US_R1206
- R3: device adafruit:R-US_R0805 -> adafruit:R-US_R1206
- R5, R6: value 1.18M -> 250R; device adafruit:R-US_R0805 -> adafruit:R-US_M0805
- R7: value 1.18M -> 3k; device adafruit:R-US_R0805 -> adafruit:R-US_M0805
- U$2: value 6-PIN-ICSPTAGCONNECT-HOLES -> 6-PIN-ICSPEASY-MSP; device LaunchFET:6-PIN-ICSPTAGCONNECT-HOLES -> LaunchFET:6-PIN-ICSPEASY-MSP
- U$3: value LTC3114 -> 1X4_HEADER; device linear:LTC3114 -> connectors:1X4_HEADER
- U$4: value DC630R-562M -> FC4L64; device connectors:DC630R-562M -> misc_passives:FC4L64
- U1: value INA209_PW_16 -> LTC1540; device TexasInstruments:INA209_PW_16 -> linear:LTC1540
- U2: value UCC2837_D_8 -> TPS70930-Q1; device TexasInstruments:UCC2837_D_8 -> TexasInstruments:TPS70930-Q1
- U3: value AD5252BRU10 -> LTC6102; device linear:AD5252BRU10 -> linear:LTC6102
Connections:
- removed net +5V: 5VRAIL.A, C17.1, JP4.10, JP4.8, U$3.PVOUT, U3.A1
- removed net 5V_ENABLE: U$3.RUN, U5.P3.2/A14*/CD14
- removed net AUTO_BAUD: U5.PJ.2/TMS/TB2OUTH/ACLK/CD8, U6.AB
- removed net BAT_CRITICAL: R7.2, U1.CRITICAL, U5.P1.1/TA0.2/TA1CLK/CDOUT/A1*/CD1/VEREF+*
- removed net BAT_OVERLIM: R6.2, U1.OVERLIMIT, U5.P1.2/TA1.1/TA0CLK/CDOUT/A2*/CD2
- removed net BAT_WARN: R5.2, U1.WARNING, U5.P3.0/A12*/CD12
- removed net CAN_H: JP4.2, U6.CANH
- removed net CAN_L: JP4.3, U6.CANL
- removed net CAN_RESET: IC1.RESET, U5.P2.7
- removed net CLK: IC1.SCK, U5.P2.4/TA1.0/UCA1CLK/A7*/CD11
- removed net EXT_XIN: IC1.CLKOUT, U5.PJ.4/XIN
- removed net GNDA: C9.2, U5.AVSS, U5.DVSS
- removed net MISO: IC1.SO, U5.P2.6/TB1.0/UCA1RXD/UCA1SOMI
- removed net MOSI: IC1.SI, U5.P2.5/TB0.0/UCA1TXD/UCA1SIMO
- removed net N$13: C10.1, U$1.LDO, U$1.PLDO
- removed net N$16: C11.2, R14.2
- removed net N$19: C16.1, R17.2, U$3.PROG
- removed net N$20: C18.1, U$3.LDO, U$3.PLDO
- removed net N$21: R2.1, R3.2, S1.2, U$1.RUN
- removed net N$22: C19.1, U$3.VC
- removed net N$23: C19.2, R18.2
- removed net N$24: U$3.FB, U3.W1
- removed net N$25: Q1.D, R25.1, U2.CS
- removed net N$26: R22.2, U5.P1.5/TB0.2/UCA0CLK/A5*/CD5
- removed net N$27: C23.1, U2.CAP
- removed net N$28: U2.FB, U3.W3
- removed net N$29: R23.1, U2.COMP
- removed net N$30: R21.2, U5.PJ.0/TDO/TB0OUTH/SMCLK/CD6
- removed net N$31: R24.2, U5.PJ.1/TDI/TCLK/TB1OUTH/MCLK/CD7
- removed net N$32: C24.1, U2.CT
- removed net N$9: C15.2, U$1.BST2
- removed net RX0BF: IC1.RX0BF, U5.P3.6/TB2.1/TB1CLK
- removed net RX1BF: IC1.RX1BF, U5.P3.5/TB1.2/CDOUT
- removed net RXINT: IC1.INT, U5.P3.7/TB2.2
- removed net RX_CAN: IC1.RXCAN, U6.R
- removed net SMBALERT: U1.SMBUSALERT, U5.P3.1/A13*/CD13
- removed net STE: IC1.CS, U5.P2.3/TA0.0/UCA1STE/A6*/CD10
- removed net TRIGGER_CONVERT: U1.CONVERT, U5.P1.0/TA0.1/DMAE0/RTCCLK/A0*/CD0/VEREF-*
- removed net TX0RTS: IC1.TX0RTS, U5.P3.4/TB1.1/TB2CLK/SMCLK
- removed net TX1RTS: IC1.TX1RTS, U5.P2.2/TB2.2/UCB0CLK/TB1.0
- removed net TX2RTS: IC1.TX2RTS, U5.PJ.3/TCK/CD9
- removed net TX_CAN: IC1.TXCAN, U6.D
- removed net VBUS: C27.1, Q1.S, U$6.1, U3.A3
- removed net VBUS_BYPASS: Q1.G, U2.VOUT, U5.P3.3/A15*/CD15
- removed net VBUS_ENABLE: C25.1, R23.2, U5.P1.3/TA1.2/UCB0STE/A3*/CD3
- removed net VCC_1: R1.1, U1.VIN+, X1-1.KL
- removed net XIN: C7.1, IC1.OSC1, Q2.2
- removed net XOUT: C8.1, IC1.OSC2, Q2.1
- new net +3V3_MCU: C3.1, C4.1, R4.2, U$2.VCC
- new net I_SENSE: R7.1, U3.OUT, U5.P3.3/A15*/CD15
- new net LED1: R24.2
- new net LED2: R21.2
- new net LED3: R22.2
- new net OB_ALERT: U$8.3, U5.P2.7
- new net T1: U4.VO, U5.P3.0/A12*/CD12
- new net VENABLE: R12.1, U1.OUT, U2.EN, U3.EN
- new net V_OUT: C7.1, JP1.1, L1.B, R13.1
- new net V_SENSE: OA1B.+, R13.2, R14.1
- new net V_SENSE_IN: OA1A.-, OA1A.OUT, U5.P3.2/A14*/CD14
- new net V_SENSE_IN_P: OA1A.+, R15.2, R16.1
- new net V_SENSE_OUT: OA1B.-, OA1B.OUT, U5.P3.1/A13*/CD13
- net +3V3: now also C11.1, C14.1, OA1A.VIN, U2.OUT, U4.+VS; no longer 100%.A, 25%.A, 3V3RAIL.A, 50%.A, 75%.A, C12.1, C28.1, C3.1, C4.1, C5.1, C9.1, IC1.VDD, JP4.7, JP4.9, R12.2, R4.2, R5.1, R6.1, R7.1, U$1.PVOUT, U$2.VCC, U1.VS+, U1.VS-, U3.AD0, U3.VDD, U3.WP*, U6.VCC
- net GND: now also C11.2, C13.2, C9.2, D1.1, D1.2, JP1.2, OA1A.GND, R12.2, R14.2, R16.2, R3.1, R7.2, U$10.E, U$12.E, U$3.1, U$3.2, U$3.3, U$3.4, U1.HYST, U1.IN-, U1.REF, U1.V-, U3.V-, U4.GND, U5.AVSS, U5.DVSS; no longer C12.2, C16.2, C17.2, C18.2, C21.2, C23.2, C24.2, C25.2, C26.2, C27.2, C28.2, C5.2, C6.2, C8.2, IC1.VSS, JP4.1, JP4.4, JP4.5, JP4.6, Q2.0, R10.2, R11.2, R13.1, R14.1, R15.1, R16.1, R17.1, R18.1, S1.1, U$1.GND, U$1.MODE, U$1.PGND, U$3.GND, U$3.MODE, U$3.PGND, U$6.2, U1.A0, U1.A1, U1.GND_2, U3.AD1, U3.B1, U3.B3, U3.DGND, U3.VSS, U6.GND, U6.RS, X1-2.KL
- net N$10: now also D1.3, FET1.S, L1.A; no longer C20.1, U$3.SW1, U$5.A
- net N$11: now also C5.1, R1.2, R10.1, U$12.C; no longer C6.1, R13.2, U$1.PROG
- net N$12: now also C6.2, R11.2, U$12.B; no longer C22.1, U$3.SW2, U$5.B
- net N$14: now also 100%.A, 25%.A, 50%.A, 75%.A; no longer C20.2, U$3.BST1
- net N$15: now also FET1.G, U$10.G; no longer C11.1, U$1.VC
- net N$17: now also C6.1, R11.1, U5.P3.7/TB2.2; no longer R12.1, R15.2, U$1.FB
- net N$18: now also C10.1, C9.1, FET1.D, R1.1, R15.1, U$10.C, U$4.1A; no longer C22.2, U$3.BST2
- net N$2: now also R5.2, U$4.2B; no longer R16.2, R3.1, S1.4
- net N$3: now also R2.1, R3.2, U1.IN+; no longer R19.2, U5.P1.4/TB0.1/UCA0STE/A4*/CD4
- net N$4: now also R6.1, U3.+IN; no longer 5VRAIL.C, R11.1
- net N$5: now also R5.1, U3.-INF, U3.-INS; no longer 3V3RAIL.C, R10.1
- net N$6: now also R6.2, U$4.1B; no longer C13.1, U$1.SW1, U$4.A
- net N$7: now also C5.2, R10.2, U$10.G1, U$10.G2; no longer C15.1, U$1.SW2, U$4.B
- net N$8: now also C8.2, U3.VREG; no longer C13.2, U$1.BST1
- net RST: now also U$8.4
- net SCL: now also U$8.2; no longer U1.SCL, U3.SCL
- net SDA: now also U$8.1; no longer U1.SDA, U3.SDA
- net UART_RX: now also U$2.TX; no longer U$2.RX
- net UART_TX: now also U$2.RX; no longer U$2.TX
- net VCC: now also C13.1, C8.1, U$11.1, U$11.2, U$11.3, U$11.4, U$4.2A, U1.V+, U2.IN, U3.V+; no longer C14.1, C21.1, C26.1, R1.2, R25.2, S1.3, U$1.PVIN, U$1.VIN, U$3.PVIN, U$3.VIN, U1.VIN-, U2.VDD
Other:
- note added: "4.3 : 1 ratio"
- note added: "50mOhm"
- note added: "Dedicated MCU supply"
- note added: "Input Voltage Sense"
- note added: "Low voltage cut off"
- note added: "Regulated Voltage Sense"
- note added: "Thermal Monitoring ---------------------------------- Place close to mosfet"
- note added: "Vbus"
- note added: "Vbus Current Sense"
- note added: "Vbus Signal"
- note added: "pwm in"
- note removed: "3.3V Rail -------------------------------- 1A max output Uses comparator to disable the rail when voltage drops below cutoff for battery type"
- note removed: "Current amp: UCB0 debug UART: UCA0 CAN_BUS: UCA1"
- note removed: "Current sense amplifier ------------------------------------------ I2C address: 10000000"
- note removed: "Cutoff Voltage selection ----------------------------------------- 0 0 : LiPo (3.2 V cutoff) 0 1 : NiMH (2V cutoff) 1 x : Default (1.1V)"
- note removed: "Digi-Pot -------------------------------- I2C Address 0x01 Dual channel pot used to adjust output voltage on two channels"
- note removed: "Low power buck-boost rail -------------------------------- 1A max adjustible votage rail output voltage adjusted through digi-pot"
- note removed: "V bus -------------------------------- High Amperage linear regulator Can be bypassed, allowing unregulated battery voltage on line"
- moved on the sheet: 100%, 25%, 50%, 75%, C1, C10, C11, C13, C14, C2, C3, C4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

Commit message: clean up schematics
Parts:
- removed 100%, 25%, 50%, 75%: (no value), adafruit:LEDCHIP-LED0603
- removed C14: 10u, adafruit:C-USC1206
- removed JP1: (no value), jumper:JP1E
- removed OA1: LMP2202, TexasInstruments:LMP2202
- removed R19, R21, R22, R24: (no value), adafruit:R-US_R0603
- removed U$10: NPN-PNP-QSZ4TR, misc_passives:NPN-PNP-QSZ4TR
- removed U$12: NPN-2SC5866TLQ, misc_passives:NPN-2SC5866TLQ
- added C12: 470n, adafruit:C-USC1206
- added T1: NPN-PNP-QSZ4TR, misc_passives:NPN-PNP-QSZ4TR
- added T2: NPN-2SC5866TLQ, misc_passives:NPN-2SC5866TLQ
- added U$1: MICROPITCH, connectors:MICROPITCH
- added U$5: MOLEX-0436500200, connectors:MOLEX-0436500200
- added U6: MSP430FR5739_DA_38, TexasInstruments:MSP430FR5739_DA_38
- C1: value 2.2n -> 10u
- C10: value 47uF -> 10u; device rcl:C-EUC1206 -> adafruit:C-USC1206
- C11: value .1uF -> 0.1u; device adafruit:C-USC0805 -> adafruit:C-USC1206
- C13: value 10u -> 2.2n
- C2: value 470n -> 10u
- C3: value 10u -> .1uF; device adafruit:C-USC1206 -> adafruit:C-USC0805
- C4: value 0.1u -> .1uF; device adafruit:C-USC1206 -> adafruit:C-USC0805
- C5, C6: value (none) -> 47uF; device adafruit:C-USC0805 -> rcl:C-EUC1206
- C8: value .1uF -> (none)
- C9: value 47uF -> (none); device rcl:C-EUC1206 -> adafruit:C-USC0805
- R1: value 10k -> 4.8M; device adafruit:R-US_M0805 -> adafruit:R-US_R1206
- R12: value 100k -> 10k; device adafruit:R-US_R1206 -> adafruit:R-US_M0805
- R13: value 10k -> 2.3k
- R14: value 2.3k -> 47k; device adafruit:R-US_M0805 -> adafruit:R-US_R1206
- R15: value 10k -> 1.18M; device adafruit:R-US_M0805 -> adafruit:R-US_R0805
- R16: value 2.3k -> 1.18M; device adafruit:R-US_M0805 -> adafruit:R-US_R0805
- R2: value 4.8M -> 1.18M
- R3: value 1.18M -> 100k
- R4: value 47k -> 250R; device adafruit:R-US_R1206 -> adafruit:R-US_M0805
- R6: value 250R -> 3k
- R7: value 3k -> 10k
- R8: value 1.18M -> 2.3k; device adafruit:R-US_R0805 -> adafruit:R-US_M0805
- R9: value 1.18M -> 10k; device adafruit:R-US_R0805 -> adafruit:R-US_M0805
- U4: value LM45_DBZ_3 -> LMP2202; device TexasInstruments:LM45_DBZ_3 -> TexasInstruments:LMP2202
- U5: value MSP430FR5739_DA_38 -> LM45_DBZ_3; device TexasInstruments:MSP430FR5739_DA_38 -> TexasInstruments:LM45_DBZ_3
- renumbered U$4 to RSENSE
Connections:
- removed net +3V3_MCU: C3.1, C4.1, R4.2, U$2.VCC
- removed net LED1: R24.2
- removed net LED2: R21.2
- removed net LED3: R22.2
- removed net N$1: 25%.C, R19.1
- removed net N$14: 100%.A, 25%.A, 50%.A, 75%.A
- removed net N$33: 50%.C, R22.1
- removed net N$34: 75%.C, R21.1
- removed net N$35: 100%.C, R24.1
- new net CLK: U$1.10, U6.P2.4/TA1.0/UCA1CLK/A7*/CD11
- new net N$13: U$1.4, U6.P2.5/TB0.0/UCA1TXD/UCA1SIMO
- new net N$16: U$1.8, U6.PJ.2/TMS/TB2OUTH/ACLK/CD8
- new net N$19: U$1.5, U6.PJ.0/TDO/TB0OUTH/SMCLK/CD6
- new net N$20: U$1.3, U6.P1.5/TB0.2/UCA0CLK/A5*/CD5
- new net N$21: U$1.1, U6.P1.4/TB0.1/UCA0STE/A4*/CD4
- new net N$22: U$1.6, U6.PJ.3/TCK/CD9
- new net N$24: U$1.2, U6.P2.6/TB1.0/UCA1RXD/UCA1SOMI
- new net PWM: C9.1, R11.1, U6.P1.3/TA1.2/UCB0STE/A3*/CD3
- new net STE: U$1.9, U6.P2.3/TA0.0/UCA1STE/A6*/CD10
- net +3V3: now also C10.1, C2.1, C4.1, R14.2, R15.1, R16.1, U$2.VCC, U4A.VIN, U5.+VS, U6.AVCC, U6.DVCC; no longer C14.1, OA1A.VIN, R8.1, R9.1, U4.+VS, U5.AVCC, U5.DVCC
- net GND: now also C12.2, C5.2, C6.2, R13.2, R2.1, R3.2, R6.2, R8.2, T1.E, T2.E, U$5.2, U4A.GND, U5.GND, U6.AVSS, U6.AVSS_2, U6.DVSS, U6.P2.2/TB2.2/UCB0CLK/TB1.0, U6.P2.7, U6.P3.4/TB1.1/TB2CLK/SMCLK, U6.P3.5/TB1.2/CDOUT, U6.P3.6/TB2.1/TB1CLK, U6.P3.7/TB2.2, U6.PJ.4/XIN, U6.PJ.5/XOUT; no longer C14.2, C3.2, C9.2, JP1.2, OA1A.GND, R12.2, R14.2, R16.2, R3.1, R7.2, U$10.E, U$12.E, U4.GND, U5.AVSS, U5.AVSS_2, U5.DVSS
- net I_SENSE: now also R6.1, U6.P3.0/A12*/CD12; no longer R7.1, U5.P3.3/A15*/CD15
- net N$11: now also C8.1, R9.2, T2.C; no longer C5.1, R1.2, U$12.C
- net N$12: now also C9.2, T2.B; no longer C6.2, U$12.B
- net N$15: now also T1.G; no longer U$10.G
- net N$17: now also U$1.7, U6.PJ.1/TDI/TCLK/TB1OUTH/MCLK/CD7; no longer C6.1, R11.1, U5.P3.7/TB2.2
- net N$18: now also C5.1, C6.1, R7.1, R9.1, T1.C; no longer C10.1, C9.1, R1.1, R15.1, U$10.C
- net N$3: now also R1.1, R2.2; no longer R2.1, R3.2
- net N$4: now also R4.1; no longer R6.1
- net N$6: now also R4.2; no longer R6.2
- net N$7: now also C8.2, T1.G1, T1.G2; no longer C5.2, U$10.G1, U$10.G2
- net N$8: now also C3.2; no longer C8.2
- net OB_ALERT: now also U6.P1.2/TA1.1/TA0CLK/CDOUT/A2*/CD2; no longer U5.P2.7
- net RST: now also C13.1, R14.1, U6.*RST/NMI/SBWTDIO; no longer C1.1, R4.1, U5.*RST/NMI/SBWTDIO
- net SCL: now also R16.2, U6.P1.7/TB1.2/UCB0SOMI/UCB0SCL/TA1.0; no longer R9.2, U5.P1.7/TB1.2/UCB0SOMI/UCB0SCL/TA1.0
- net SDA: now also R15.2, U6.P1.6/TB1.1/UCB0SIMO/UCB0SDA/TA0.0; no longer R8.2, U5.P1.6/TB1.1/UCB0SIMO/UCB0SDA/TA0.0
- net T1: now also U5.VO, U6.P3.2/A14*/CD14; no longer U4.VO, U5.P3.0/A12*/CD12
- net TEST: now also U6.TEST/SBWTCK; no longer U5.TEST/SBWTCK
- net UART_RX: now also U6.P2.1/TB2.1/UCA0RXD/UCA0SOMI/TB0.0; no longer U5.P2.1/TB2.1/UCA0RXD/UCA0SOMI/TB0.0
- net UART_TX: now also U6.P2.0/TB2.0/UCA0TXD/UCA0SIMO/TB0CLK/ACLK; no longer U5.P2.0/TB2.0/UCA0TXD/UCA0SIMO/TB0CLK/ACLK
- net VCC: now also C1.1, C3.1, R1.2; no longer C13.1, C8.1, R2.2
- net VCORE: now also C12.1, U6.VCORE; no longer C2.1, U5.VCORE
- net VENABLE: now also R3.1; no longer R12.1
- net V_OUT: now also R12.1, U$5.1; no longer JP1.1, R13.1
- net V_SENSE: now also R12.2, R13.1, U4B.+; no longer OA1B.+, R13.2, R14.1
- net V_SENSE_IN: now also U4A.-, U4A.OUT, U6.P3.1/A13*/CD13; no longer OA1A.-, OA1A.OUT, U5.P3.2/A14*/CD14
- net V_SENSE_IN_P: now also R7.2, R8.1, U4A.+; no longer OA1A.+, R15.2, R16.1
- net V_SENSE_OUT: now also U4B.-, U4B.OUT, U6.P3.3/A15*/CD15; no longer OA1B.-, OA1B.OUT, U5.P3.1/A13*/CD13
Other:
- note added: "Aux port"
- note added: "I2C pull up"
- note added: "ICSP"
- note added: "MCU"
- note added: "MCU conditioning"
- note added: "Mosfet and driver"
- note added: "Regulated Output"
- note removed: "pwm in"
- moved on the sheet: C1, C10, C11, C13, C2, C3, C4, C5, C6, C7, C8, C9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
